Commit message: Reinforce D6.2 floor panels with four distributed fixings
Anchor the printed seam beam at both ends, add tapered underside ribs, and retain battery and computer access. Treat 10 kg as a soft vehicle target and recalculate the 10 kg cargo cases through a 10.5 kg vehicle envelope. Regenerate CAD, print files, BOM, screenshots, URDF and the verified MuJoCo motion GIF.

File: sim/isaac_sim/amr_d62.urdf (robot description, URDF)
Before this commit: robot amr_d61, 5 links, 4 joints
Links:
- link base_link: mass 8.87086255317 -> 9.11550857337; geometry collision box size=0.0032 0.1 0.015; collision box size=0.0032 0.1 0.015

File: sim/isaac_sim/amr_d62_payload_10kg.urdf (robot description, URDF)
Before this commit: robot amr_d61_payload_10kg, 6 links, 5 joints
Links:
- link base_link: mass 8.87086255317 -> 9.11550857337; geometry collision box size=0.0032 0.1 0.015; collision box size=0.0032 0.1 0.015
