Commit message: Extend D6.3 floor corners and remove auxiliary flat gussets
Keep eight independent HBLFSN6 frame joints and four fixings per floor panel. Remove four notched flat plates and their eight fastener sets after detecting half-supported washer seats. Update CAD, print files, BOM, reviews, screenshots and simulation assets; retain explicit limits on physical joint stiffness qualification.

File: sim/isaac_sim/amr_d63.urdf (robot description, URDF)
Before this commit: robot amr_d62, 5 links, 4 joints
Links:
- link base_link: mass 9.11550857337 -> 8.9931237619

File: sim/isaac_sim/amr_d63_payload_10kg.urdf (robot description, URDF)
Before this commit: robot amr_d62_payload_10kg, 6 links, 5 joints
Links:
- link base_link: mass 9.11550857337 -> 8.9931237619
