Commit message: Replace PLA floor countersinks with plain M4 holes and large washers

File: sim/isaac_sim/amr_d64.urdf (robot description, URDF)
Before this commit: robot amr_d63_payload_10kg, 6 links, 5 joints
Links:
- removed link payload_link
- link base_link: mass 8.9931237619 -> 9.00487528613; geometry collision box size=0.0032 0.1 0.015; collision box size=0.0032 0.1 0.015
Joints:
- removed joint payload_fixed_joint

File: sim/isaac_sim/amr_d64_payload_10kg.urdf (robot description, URDF)
Before this commit: robot amr_d63, 5 links, 4 joints
Links:
- added link payload_link, mass 10; collision box size=0.2 0.2 0.16; visual box size=0.2 0.2 0.16
- link base_link: mass 8.9931237619 -> 9.00487528613; geometry collision box size=0.0032 0.1 0.015; collision box size=0.0032 0.1 0.015
Joints:
- added joint payload_fixed_joint: type fixed, parent base_link, child payload_link, origin xyz=-0.09 0 0.26265 rpy=0 0 0
