Commit message: Cover computer floor fasteners with a removable PLA barrier
Add a continuous 2 mm cover over the four M4 heads and washers, retain aligned case supports, and distinguish the unselected PCB mount from the contact barrier. Update saved CAD, screenshots, printable parts, mass and cost ledgers, floor analysis, and simulation artifacts.

File: sim/isaac_sim/amr_d65.urdf (robot description, URDF)
Before this commit: robot amr_d64_payload_10kg, 6 links, 5 joints
Links:
- removed link payload_link
- link base_link: mass 9.00487528613 -> 9.04346426469; geometry collision box size=0.0032 0.1 0.015; collision box size=0.0032 0.1 0.015
Joints:
- removed joint payload_fixed_joint

File: sim/isaac_sim/amr_d65_payload_10kg.urdf (robot description, URDF)
Before this commit: robot amr_d64, 5 links, 4 joints
Links:
- added link payload_link, mass 10; collision box size=0.2 0.2 0.16; visual box size=0.2 0.2 0.16
- link base_link: mass 9.00487528613 -> 9.04346426469; geometry collision box size=0.0032 0.1 0.015; collision box size=0.0032 0.1 0.015
Joints:
- added joint payload_fixed_joint: type fixed, parent base_link, child payload_link, origin xyz=-0.09 0 0.26265 rpy=0 0 0
